Commit message: [WIP]

File: src/urdf/leo_arm_sim.urdf.xacro (robot description, xacro)
@@ -7,4 +7,7 @@
   <xacro:include filename="$(find leo_description)/urdf/macros.xacro"/>
   <xacro:include filename="$(find arm_integration)/urdf/mobile_px100.urdf.xacro"/>
+  <xacro:leo_sim robot_ns="$(arg robot_ns)"
+                 fixed="$(arg fixed)"
+                 mecanum_wheels="$(arg mecanum_wheels)"/>
 <joint name="arm_joint" type="fixed">
 <origin xyz="0.043 0 -0.001"/>
@@ -12,6 +15,3 @@
 <child link="mobile_px100/base_link"/>
 </joint>
-  <xacro:leo_sim robot_ns="$(arg robot_ns)"
-                 fixed="$(arg fixed)"
-                 mecanum_wheels="$(arg mecanum_wheels)"/>
 </robot>

File: src/urdf/mobile_px100.urdf.xacro (robot description, xacro)
@@ -16,5 +16,6 @@
   <xacro:arg name="external_urdf_loc"               default=""/>
   <xacro:arg name="hardware_type"                   default="actual"/>
-  <xacro:property name="mesh_directory"             value="$(find interbotix_xsarm_descriptions)/meshes/${robot_model}_meshes"/>
+  <!-- <xacro:property name="mesh_directory"             value="$(find interbotix_xsarm_descriptions)/meshes/${robot_model}_meshes"/> -->
+  <xacro:property name="mesh_directory"             value="package://interbotix_xsarm_descriptions/meshes/${robot_model}_meshes"/>
   <xacro:property name="urdf_loc"                   value="$(arg external_urdf_loc)"/>
   <xacro:property name="hardware_type"              value="$(arg hardware_type)"/>
